Commit message: Fix UR5 Robotiq gripper closure

File: assets/robots/ur5e/ur5e_robotiq_2f_85.urdf (robot description, URDF)
Before this commit: robot ur5e_robotiq_2f_85, 22 links, 21 joints
Joints:
- joint finger_joint: axis (none) -> 1 0 0; limit (none) -> lower=0 upper=0.8 effort=1000 velocity=2.0; type fixed -> revolute
- joint left_inner_finger_joint: axis (none) -> 1 0 0; limit (none) -> lower=-0.8757 upper=0 effort=1000 velocity=2.0; mimic (none) -> joint=finger_joint multiplier=-1 offset=0; type fixed -> revolute
- joint left_inner_finger_pad_joint: origin xyz=0 -0.0220203446692936 0.03242 rpy=0 0 0 -> xyz=0 -0.0320 0.03242 rpy=0.20 0 0
- joint left_inner_knuckle_joint: axis (none) -> 1 0 0; limit (none) -> lower=0 upper=0.8757 effort=1000 velocity=2.0; mimic (none) -> joint=finger_joint multiplier=1 offset=0; type fixed -> revolute
- joint right_inner_finger_joint: axis (none) -> 1 0 0; limit (none) -> lower=-0.8757 upper=0 effort=1000 velocity=2.0; mimic (none) -> joint=finger_joint multiplier=-1 offset=0; type fixed -> revolute
- joint right_inner_finger_pad_joint: origin xyz=0 -0.0220203446692936 0.03242 rpy=0 0 0 -> xyz=0 -0.0320 0.03242 rpy=0.20 0 0
- joint right_inner_knuckle_joint: axis (none) -> 1 0 0; limit (none) -> lower=0 upper=0.8757 effort=1000 velocity=2.0; mimic (none) -> joint=finger_joint multiplier=1 offset=0; type fixed -> revolute
- joint right_outer_knuckle_joint: axis (none) -> 1 0 0; limit (none) -> lower=0 upper=0.81 effort=1000 velocity=2.0; mimic (none) -> joint=finger_joint multiplier=1 offset=0; type fixed -> revolute

Commit message: Rebuild UR5e Robotiq model and Berkeley TCP

File: assets/robots/ur5e/ur5e_robotiq_2f_85.urdf (robot description, URDF)
Before this commit: robot ur5e_robotiq_2f_85, 22 links, 21 joints
Links:
- link left_inner_finger: mass 0.01 -> 0.0125222; geometry collision mesh filename=robotiq_2f_85/meshes/menagerie_v4/follower.stl scale=1 1 1; collision mesh filename=robotiq_2f_85/meshes/menagerie_v4/tongue.stl scale=1 1 1
- link left_inner_finger_pad: mass 0.01 -> 0.0035; geometry collision box size=0.004 0.022 0.01875; collision box size=0.004 0.022 0.01875
- link left_inner_knuckle: mass 0.01 -> 0.0221642; geometry collision mesh filename=robotiq_2f_85/meshes/menagerie_v4/spring_link.stl scale=1 1 1; visual mesh filename=robotiq_2f_85/meshes/menagerie_v4/spring_link.stl scale=1 1 1
- link left_outer_finger: mass 0.01 -> 0.0140974; geometry collision mesh filename=robotiq_2f_85/meshes/menagerie_v4/coupler.stl scale=1 1 1; visual mesh filename=robotiq_2f_85/meshes/menagerie_v4/coupler.stl scale=1 1 1
- link left_outer_knuckle: mass 0.01 -> 0.00899563; geometry collision mesh filename=robotiq_2f_85/meshes/menagerie_v4/driver.stl scale=1 1 1; visual mesh filename=robotiq_2f_85/meshes/menagerie_v4/driver.stl scale=1 1 1
- link right_inner_finger: mass 0.01 -> 0.0125222; geometry collision mesh filename=robotiq_2f_85/meshes/menagerie_v4/follower.stl scale=1 1 1; collision mesh filename=robotiq_2f_85/meshes/menagerie_v4/tongue.stl scale=1 1 1
- link right_inner_finger_pad: mass 0.01 -> 0.0035; geometry collision box size=0.004 0.022 0.01875; collision box size=0.004 0.022 0.01875
- link right_inner_knuckle: mass 0.01 -> 0.0221642; geometry collision mesh filename=robotiq_2f_85/meshes/menagerie_v4/spring_link.stl scale=1 1 1; visual mesh filename=robotiq_2f_85/meshes/menagerie_v4/spring_link.stl scale=1 1 1
- link right_outer_finger: mass 0.01 -> 0.0140974; geometry collision mesh filename=robotiq_2f_85/meshes/menagerie_v4/coupler.stl scale=1 1 1; visual mesh filename=robotiq_2f_85/meshes/menagerie_v4/coupler.stl scale=1 1 1
- link right_outer_knuckle: mass 0.01 -> 0.00899563; geometry collision mesh filename=robotiq_2f_85/meshes/menagerie_v4/driver.stl scale=1 1 1; visual mesh filename=robotiq_2f_85/meshes/menagerie_v4/driver.stl scale=1 1 1
- link robotiq_arg2f_base_link: mass 0.01 -> 0.777441; geometry collision mesh filename=robotiq_2f_85/meshes/menagerie_v4/base.stl scale=1 1 1; collision mesh filename=robotiq_2f_85/meshes/menagerie_v4/base_coupling.stl scale=1 1 1
- link tool0: geometry collision cylinder length=0.06 radius=0.018; visual cylinder length=0.06 radius=0.018
Joints:
- joint finger_joint: axis 1 0 0 -> 0 0 1; limit lower=0 upper=0.8 effort=1000 velocity=2.0 -> lower=0 upper=0.9 effort=5 velocity=2; origin xyz=0 -0.0306011 0.054904 rpy=0 0 3.141592653589793 -> xyz=-0.0306011 0.00475 0.0657045 rpy=-1.5707963267948966 0 0
- joint left_inner_finger_joint: axis 1 0 0 -> 0 0 1; limit lower=-0.8757 upper=0 effort=1000 velocity=2.0 -> lower=0 upper=0.9 effort=5 velocity=2; mimic joint=finger_joint multiplier=-1 offset=0 -> joint=finger_joint multiplier=1 offset=0; origin xyz=0 0.0061 0.0471 rpy=0 0 0 -> xyz=-0.0382079 -0.0425003 0.00295 rpy=-3.141592653589793 0 0.0000380462; parent left_outer_finger -> left_inner_knuckle
- joint left_inner_finger_pad_joint: origin xyz=0 -0.0320 0.03242 rpy=0.20 0 0 -> xyz=-0.0377897 -0.103916 -0.0091 rpy=-1.5707963267948966 0 0
- joint left_inner_knuckle_joint: axis 1 0 0 -> 0 0 1; limit lower=0 upper=0.8757 effort=1000 velocity=2.0 -> lower=0 upper=0.9 effort=5 velocity=2; origin xyz=0 -0.0127 0.06142 rpy=0 0 3.141592653589793 -> xyz=-0.0127 -0.012 0.07222 rpy=-1.5707963267948966 0 0
- joint left_outer_finger_joint: origin xyz=0 0.0315 -0.0041 rpy=0 0 0 -> xyz=-0.0314249 0.00453223 -0.0102 rpy=0 0 3.141592653589793
- joint right_inner_finger_joint: axis 1 0 0 -> 0 0 1; limit lower=-0.8757 upper=0 effort=1000 velocity=2.0 -> lower=0 upper=0.9 effort=5 velocity=2; mimic joint=finger_joint multiplier=-1 offset=0 -> joint=finger_joint multiplier=1 offset=0; origin xyz=0 0.0061 0.0471 rpy=0 0 0 -> xyz=-0.0382079 -0.0425003 0.00295 rpy=-3.141592653589793 0 0; parent right_outer_finger -> right_inner_knuckle
- joint right_inner_finger_pad_joint: origin xyz=0 -0.0320 0.03242 rpy=0.20 0 0 -> xyz=-0.0377897 -0.103916 -0.0091 rpy=-1.5707963267948966 0 0
- joint right_inner_knuckle_joint: axis 1 0 0 -> 0 0 1; limit lower=0 upper=0.8757 effort=1000 velocity=2.0 -> lower=0 upper=0.9 effort=5 velocity=2; origin xyz=0 0.0127 0.06142 rpy=0 0 0 -> xyz=0.0127 0.012 0.07222 rpy=-1.5707963267948966 0 3.141592653589793
- joint right_outer_finger_joint: origin xyz=0 0.0315 -0.0041 rpy=0 0 0 -> xyz=-0.0314249 0.00453223 -0.0102 rpy=0 0 3.141592653589793
- joint right_outer_knuckle_joint: axis 1 0 0 -> 0 0 1; limit lower=0 upper=0.81 effort=1000 velocity=2.0 -> lower=0 upper=0.9 effort=5 velocity=2; origin xyz=0 0.0306011 0.054904 rpy=0 0 0 -> xyz=0.0306011 -0.00475 0.0657045 rpy=-1.5707963267948966 0 3.141592653589793
- joint tool0_to_robotiq_arg2f_base_link: origin xyz=0 0 0 rpy=0 0 0 -> xyz=0 0 0 rpy=0 0 1.5707963267948966
